File: sources/adafruit-music-maker/kicad/Adafruit-Music-Maker-MP3-Shield.sch (KiCad schematic (older format))
At the start: 88 parts, among them CN1 2908-05WB-M6, SW2 SPST_TACT-EVQQ2, U1 VS1053B, U2 AP7312-1833W6-7, U4 TS2012, U5 74HC4050D, X1 19621, Y1 ABM8G-12.288MHZ-4Y-T3

Commit message: Got stuck in KiCAD importer - not linking to symbols
Parts:
- removed SYM?: ARDUINO_R3_ICSP, symbol Adafruit-Music-Maker-MP3-Shield-eagle-import:ARDUINO_R3_ICSP
Changed lines of the file:
@@
 Wire Notes Line
 	1300 6000 16200 6000
-$Comp
-L Adafruit-Music-Maker-MP3-Shield-eagle-import:ARDUINO_R3_ICSP SYM?
-U 1 1 617F0C29
-P 8800 9700
-F 0 "SYM?" H 8800 9700 50  0001 C CNN
-F 1 "ARDUINO_R3_ICSP" H 8800 9700 50  0001 C CNN
-F 2 "" H 8800 9700 50  0001 C CNN
-F 3 "" H 8800 9700 50  0001 C CNN
-	1    8800 9700
-	1    0    0    -1
-$EndComp
 $EndSCHEMATC
